File: Hardware/rv32i/mem.brd (EAGLE design)
At the start: 99 x 98.7 mm, 27 parts, among them IC1 IS61C5128AS-25QLI, IC10 SN74HC138PWR, IC2 IS61C5128AS-25QLI, IC3 IS61C5128AS-25QLI, IC4 IS61C5128AS-25QLI, IC5 IS61C5128AS-25QLI, IC6 IS61C5128AS-25QLI, IC7 IS61C5128AS-25QLI, IC8 IS61C5128AS-25QLI, IC9 SN74HC138PWR

Commit message: Memory pcb layout
Parts:
- added R10, R11, R12, R13, R14, R15, R16, R17, R18, R19, R20, R21, R22, R23, R24, R25, R26, R27, R28, R29, R3, R30, R31, R32, R33, R34, R35, R36, R37, R38, R39, R4, R40, R41, R42, R43, R44, R45, R46, R47, R48, R49, R5, R50, R51, R52, R53, R54, R55, R56, R57, R58, R59, R6, R60, R61, R62, R63, R64, R7, R8, R9: RC0603FR-0710KL, RC0603FR-0710KL:RESC1608X55N
- moved JP6 353.1 mm to (91.4, 49.5), turned to 90 degrees
- moved JP4 242.6 mm to (96.5, 49.5), turned to 90 degrees
- moved JP1 201.0 mm to (72.4, 3.81)
- moved JP2 200.1 mm to (72.4, 8.89)
- moved JP3 196.1 mm to (73.7, 90.2), turned to 180 degrees
- moved JP5 193.1 mm to (73.7, 95.2), turned to 180 degrees
- moved R1 162.1 mm to (54.6, 15.2), turned to 90 degrees
- moved IC9 139.2 mm to (39.4, 5.08)
- moved R2 118.8 mm to (57.1, 15.2), turned to 90 degrees
- moved IC8 77.0 mm to (12.7, 33.0)
- moved C4 61.4 mm to (-83.8, 91.4)
- moved IC10 61.1 mm to (39.4, 90.2), turned to 180 degrees
- moved IC2 53.8 mm to (74.9, 33.0)
- moved C7 41.3 mm to (-63.5, 94.0)
- moved C8 41.3 mm to (-83.8, 94.0)
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Connections:
- net B0_A0: now also R1.1
- net B0_A1: now also R2.1
- net B0_A10: now also R11.1
- net B0_A11: now also R12.1
- net B0_A12: now also R13.1
- net B0_A13: now also R14.1
- net B0_A14: now also R15.1
- net B0_A15: now also R17.1
- net B0_A16: now also R16.1
- net B0_A17: now also R18.1
- net B0_A18: now also R19.1
- net B0_A19: now also R20.1
- net B0_A2: now also R3.1
- net B0_A20: now also R21.1
- net B0_A21: now also R22.1
- net B0_A22: now also R23.1
- net B0_A23: now also R24.1
- net B0_A24: now also R26.1
- net B0_A25: now also R25.1
- net B0_A26: now also R27.1
- net B0_A27: now also R28.1
- net B0_A28: now also R29.1
- net B0_A29: now also R30.1
- net B0_A3: now also R4.1
- net B0_A30: now also R31.1
- net B0_A31: now also R32.1
- net B0_A4: now also R5.1
- net B0_A5: now also R6.1
- net B0_A6: now also R7.1
- net B0_A7: now also R8.1
- net B0_A8: now also R9.1
- net B0_A9: now also R10.1
- net B1_A0: now also R33.1
- net B1_A1: now also R34.1
- net B1_A10: now also R43.1
- net B1_A11: now also R44.1
- net B1_A12: now also R45.1
- net B1_A13: now also R46.1
- net B1_A14: now also R47.1
- net B1_A15: now also R49.1
- net B1_A16: now also R48.1
- net B1_A17: now also R50.1
- net B1_A18: now also R51.1
- net B1_A19: now also R52.1
- net B1_A2: now also R35.1
- net B1_A20: now also R53.1
- net B1_A21: now also R54.1
- net B1_A22: now also R55.1
- net B1_A23: now also R56.1
- net B1_A24: now also R58.1
- net B1_A25: now also R57.1
- net B1_A26: now also R59.1
- net B1_A27: now also R60.1
- net B1_A28: now also R61.1
- net B1_A29: now also R62.1
- net B1_A3: now also R36.1
- net B1_A30: now also R63.1
- net B1_A31: now also R64.1
- net B1_A4: now also R37.1
- net B1_A5: now also R38.1
- net B1_A6: now also R39.1
- net B1_A7: now also R40.1
- net B1_A8: now also R41.1
- net B1_A9: now also R42.1
- net GND: now also R10.2, R11.2, R12.2, R13.2, R14.2, R15.2, R16.2, R17.2, R18.2, R19.2, R20.2, R21.2, R22.2, R23.2, R24.2, R25.2, R26.2, R27.2, R28.2, R29.2, R3.2, R30.2, R31.2, R32.2, R33.2, R34.2, R35.2, R36.2, R37.2, R38.2, R39.2, R4.2, R40.2, R41.2, R42.2, R43.2, R44.2, R45.2, R46.2, R47.2, R48.2, R49.2, R5.2, R50.2, R51.2, R52.2, R53.2, R54.2, R55.2, R56.2, R57.2, R58.2, R59.2, R6.2, R60.2, R61.2, R62.2, R63.2, R64.2, R7.2, R8.2, R9.2
Routing:
- net B0_A10: track 10.8 -> 0.00 mm, vias 1 -> 0
- net B0_A11: track 9.35 -> 0.00 mm, vias 1 -> 0
- net B0_A13: track 6.66 -> 0.00 mm, vias 1 -> 0
- net B0_A9: track 6.66 -> 0.00 mm, vias 1 -> 0
- net B0_A0: track 6.66 -> 0.00 mm, vias 1 -> 0
- net B0_A7: track 6.51 -> 0.00 mm, vias 1 -> 0
- net B0_A18: track 6.02 -> 0.00 mm, vias 1 -> 0
- net B0_A8: track 5.76 -> 0.00 mm, vias 1 -> 0
- net B0_A1: track 5.76 -> 0.00 mm, vias 1 -> 0
- net B0_A6: track 5.61 -> 0.00 mm, vias 1 -> 0
- net B0_A2: track 4.86 -> 0.00 mm, vias 1 -> 0
- net B0_A5: track 4.71 -> 0.00 mm, vias 1 -> 0
- net B0_A17: track 4.71 -> 0.00 mm, vias 1 -> 0
- net B0_A4: track 4.34 -> 0.00 mm, vias 1 -> 0
- net B0_A3: track 3.97 -> 0.00 mm, vias 1 -> 0
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Other:
- board size 99 x 98.7 mm -> 101.6 x 98.7 mm

Commit message: Update memory schematic & parts
Parts:
- added C10: CC0603KRX7R9BB104, CC0603KRX7R9BB104:CAPC1608X90N
- moved R45 196.5 mm to (49.5, 83.8), turned to 270 degrees
- moved R60 194.8 mm to (53.3, 86.4), turned to 270 degrees
- moved R40 183.7 mm to (62.2, 83.8), turned to 270 degrees
- moved R46 182.3 mm to (47.0, 83.8), turned to 270 degrees
- moved R55 182.1 mm to (66.0, 86.4), turned to 270 degrees
- moved R61 180.8 mm to (50.8, 86.4), turned to 270 degrees
- moved R35 171.0 mm to (74.9, 83.8), turned to 270 degrees
- moved R41 169.6 mm to (59.7, 83.8), turned to 270 degrees
- moved R50 169.4 mm to (78.7, 86.4), turned to 270 degrees
- moved R56 168.2 mm to (63.5, 86.4), turned to 270 degrees
- moved R62 167.0 mm to (48.3, 86.4), turned to 270 degrees
- moved R47 166.1 mm to (45.7, 86.4), turned to 270 degrees
- moved R36 156.9 mm to (72.4, 83.8), turned to 270 degrees
- moved R57 156.8 mm to (58.4, 86.4), turned to 270 degrees
- moved R63 155.8 mm to (44.5, 83.8), turned to 270 degrees
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Connections:
- net GND: now also C10.1
- net VCC: now also C10.2
Routing:
- net VCC: track 0.00 -> 440.7 mm, vias 0 -> 1
- net OE: track 0.00 -> 182.9 mm
- net WE: track 0.00 -> 153.0 mm, vias 0 -> 2
- net B0_A0: track 0.00 -> 146.4 mm, vias 0 -> 1
- net B1_A14: track 0.00 -> 135.4 mm
- net B1_A18: track 0.00 -> 121.8 mm, vias 0 -> 3
- net B1_A0: track 0.00 -> 119.6 mm, vias 0 -> 2
- net B1_D0: track 0.00 -> 118.7 mm, vias 0 -> 1
- net B1_D1: track 0.00 -> 118.4 mm, vias 0 -> 1
- net B0_A14: track 0.00 -> 117.7 mm, vias 0 -> 2
- net B0_A12: track 0.00 -> 117.7 mm, vias 0 -> 3
- net B1_A1: track 0.00 -> 116.5 mm, vias 0 -> 2
- net B0_D5: track 0.00 -> 114.1 mm, vias 0 -> 1
- net B0_A15: track 0.00 -> 113.8 mm, vias 0 -> 2
- net B0_A18: track 0.00 -> 112.9 mm, vias 0 -> 3
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Other:
- board size 101.6 x 98.7 mm -> 100.3 x 98.7 mm

Commit message: Finish memory pcb & assembly files
Parts:
- moved C10 10.9 mm to (35.9, 16.8), turned to 90 degrees
- moved IC9 8.64 mm to (31.1, 15.2)
- moved IC10 8.01 mm to (30.8, 84.5)
- moved C1 3.88 mm to (26.0, 82.9), turned to 270 degrees
- moved C8 0.90 mm to (18.4, 73.0)
- moved C2 0.64 mm to (80.0, 73.0)
- moved C5 0.64 mm to (39.4, 73.0)
- moved C6 0.64 mm to (59.7, 73.0)
Routing:
- net CE7: track 0.00 -> 84.0 mm, vias 0 -> 2
- net VCC: track 440.7 -> 524.3 mm, vias 1 -> 3
- net CE1: track 0.00 -> 71.5 mm, vias 0 -> 2
- net CE6: track 0.00 -> 63.0 mm, vias 0 -> 2
- net CE2: track 0.00 -> 52.5 mm, vias 0 -> 2
- net B0_A0: track 146.4 -> 96.1 mm, vias 1 -> 2
- net B0_A20: track 8.78 -> 58.7 mm
- net B1_A20: track 8.78 -> 56.0 mm, vias 0 -> 1
- net B0_A19: track 8.78 -> 51.7 mm
- net B1_A19: track 8.78 -> 51.7 mm, vias 0 -> 1
- net CE5: track 0.00 -> 42.1 mm, vias 0 -> 2
- net CE4: track 0.00 -> 36.3 mm, vias 0 -> 2
- net B1_A14: track 135.4 -> 99.8 mm, vias 0 -> 1
- net CE3: track 0.00 -> 34.1 mm, vias 0 -> 2
- net CE0: track 0.00 -> 30.3 mm, vias 0 -> 2
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- added copper zone on layer 1, net GND
- added copper zone on layer 16, net GND
Other:
- outline, holes or cut-outs redrawn
- board text added: "rv32i ram module v1.0"
