File: Hardware/rv32i/alu.brd (EAGLE design)
At the start: 98.7 x 99 mm, 81 parts, among them IC1 SN74HCS86DR, IC10 SN74HCS86DR, IC11 SN74HCS86DR, IC12 SN74HCS86DR, IC13 SN74HCS86DR, IC14 SN74HCS86DR, IC15 SN74HCS86DR, IC16 SN74HCS86DR, IC17 SN74HCS86DR, IC18 SN74HCS86DR, IC19 SN74HCS86DR, IC2 SN74HCS86DR, IC20 SN74HCS86DR, IC21 SN74HCS86DR, IC22 SN74HCS86DR, IC23 SN74HCS86DR, IC24 SN74HCS86DR, IC25 SN74ACT08D, IC26 SN74ACT08D, IC27 SN74ACT08D, IC28 SN74ACT08D, IC29 SN74ACT08D, IC3 SN74HCS86DR, IC30 SN74ACT08D, IC31 SN74ACT08D, IC32 SN74ACT08D, IC33 SN74ACT08D, IC34 SN74ACT08D, IC35 SN74ACT08D, IC36 SN74ACT08D, IC37 SN74ACT08D, IC38 SN74ACT08D, IC39 SN74ACT08D, IC4 SN74HCS86DR, IC40 SN74ACT08D, IC41 SN74HCS32DR, IC42 SN74HCS32DR, IC43 SN74HCS32DR, IC44 SN74HCS32DR, IC45 SN74HCS32DR, IC46 SN74HCS32DR, IC47 SN74HCS32DR, IC48 SN74HCS32DR, IC5 SN74HCS86DR, IC6 SN74HCS86DR, IC7 SN74HCS86DR, IC8 SN74HCS86DR, IC9 SN74HCS86DR

Commit message: ALU Headers & Timing Gates
Parts:
- added JP2, JP3, JP4, JP5, JP6: (no value), pinhead:2X20
- added R33, R34, R35, R36, R37, R38, R39, R40, R41, R42, R43, R44, R45, R46, R47, R48, R49, R50, R51, R52, R53, R54, R55, R56, R57, R58, R59, R60, R61, R62, R63, R64: RC0603FR-0710KL, RC0603FR-0710KL:RESC1608X55N
- moved R1 181.5 mm to (-163.8, -196.8)
- moved R3 176.9 mm to (-163.8, -199.4)
- moved R2 173.6 mm to (-146.1, -196.8)
- moved R5 172.5 mm to (-163.8, -201.9)
- moved R4 169.7 mm to (-146.1, -199.4)
- moved R7 168.4 mm to (-163.8, -204.5)
- moved R6 166.2 mm to (-146.1, -201.9)
- moved R9 164.5 mm to (-163.8, -207.0)
- moved R8 163.0 mm to (-146.1, -204.5)
- moved R11 161.0 mm to (-163.8, -209.6)
- moved R10 160.1 mm to (-146.1, -207.0)
- moved R13 157.8 mm to (-163.8, -212.1)
- moved R12 157.5 mm to (-146.1, -209.6)
- moved R14 155.4 mm to (-146.1, -212.1)
- moved R15 155.0 mm to (-163.8, -214.6)
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Connections:
- removed net N$10: JP1.22, R26.1
- removed net N$11: JP1.24, R25.1
- removed net N$12: JP1.26, R17.1
- removed net N$13: JP1.28, R18.1
- removed net N$14: JP1.30, R19.1
- removed net N$16: JP1.32, R20.1
- removed net N$17: JP1.34, R22.1
- removed net N$18: JP1.36, R21.1
- removed net N$19: JP1.38, R23.1
- removed net N$2: JP1.10, R31.1
- removed net N$4: JP1.12, R32.1
- removed net N$5: JP1.14, R30.1
- removed net N$6: JP1.16, R29.1
- removed net N$7: JP1.18, R28.1
- removed net N$9: JP1.20, R27.1
- new net D1_B0: JP2.5, JP3.5, R1.1
- new net D2_B0: JP1.5, JP4.5, R33.1
- new net SUM_B0: JP5.5, JP6.5
- new net VCC: JP1.1, JP1.2, JP1.39, JP1.40, JP2.1, JP2.2, JP2.39, JP2.40, JP3.1, JP3.2, JP3.39, JP3.40, JP4.1, JP4.2, JP4.39, JP4.40, JP5.1, JP5.2, JP5.39, JP5.40, JP6.1, JP6.2, JP6.39, JP6.40
- net D1_B1: now also JP2.7, JP3.7, R2.1; no longer JP1.40, R24.1
- net D1_B10: now also JP2.25, JP3.25, R11.1, R12.1; no longer JP1.31, R4.2
- net D1_B11: now also JP2.27, JP3.27
- net D1_B12: now also JP2.29, JP3.29, R13.1; no longer JP1.29, R3.2
- net D1_B13: now also JP2.31, JP3.31, R14.1
- net D1_B14: now also JP2.33, JP3.33, R15.1; no longer JP1.27, R2.2
- net D1_B15: now also JP2.35, JP3.35, R17.1
- net D1_B16: now also JP2.6, JP3.6, R16.1; no longer JP1.25, R1.2
- net D1_B17: now also JP2.8, JP3.8, R18.1
- net D1_B18: now also JP2.10, JP3.10, R19.1; no longer JP1.23, R9.2
- net D1_B19: now also JP2.12, JP3.12, R20.1
- net D1_B2: now also JP2.9, JP3.9, R3.1; no longer JP1.39, R8.2
- net D1_B20: now also JP2.14, JP3.14, R21.1; no longer JP1.21, R10.2
- net D1_B21: now also JP2.16, JP3.16, R22.1
- net D1_B22: now also JP2.18, JP3.18, R23.1; no longer JP1.19, R11.2
- net D1_B23: now also JP2.20, JP3.20, R24.1
- net D1_B24: now also JP2.22, JP3.22, R26.1; no longer JP1.17, R12.2
- net D1_B25: now also JP2.24, JP3.24, R25.1
- net D1_B26: now also JP2.26, JP3.26, R27.1; no longer JP1.15, R13.2
- net D1_B27: now also JP2.28, JP3.28, R28.1
- net D1_B28: now also JP2.30, JP3.30, R29.1; no longer JP1.13, R14.2
- net D1_B29: now also JP2.32, JP3.32, R30.1
- net D1_B3: now also JP2.11, JP3.11, R4.1
- net D1_B30: now also JP2.34, JP3.34, R31.1; no longer JP1.11, R16.2
- net D1_B31: now also JP2.36, JP3.36, R32.1
- net D1_B32: no longer JP1.9, R15.2
- net D1_B4: now also JP2.13, JP3.13, R5.1; no longer JP1.37, R7.2
- net D1_B5: now also JP2.15, JP3.15, R6.1
- net D1_B6: now also JP2.17, JP3.17, R7.1; no longer JP1.35, R5.2
- net D1_B7: now also JP2.19, JP3.19, R8.1
- net D1_B8: now also JP2.21, JP3.21, R9.1; no longer JP1.33, R6.2
- net D1_B9: now also JP2.23, JP3.23, R10.1
- net D2_B1: now also JP1.7, JP4.7, R34.1
- net D2_B10: now also JP1.25, JP4.25, R43.1
- net D2_B11: now also JP1.27, JP4.27, R44.1
- net D2_B12: now also JP1.29, JP4.29, R45.1
- net D2_B13: now also JP1.31, JP4.31, R46.1
- net D2_B14: now also JP1.33, JP4.33, R47.1
- net D2_B15: now also JP1.35, JP4.35, R49.1
- net D2_B16: now also JP1.6, JP4.6, R48.1
- net D2_B17: now also JP1.8, JP4.8, R50.1
- net D2_B18: now also JP1.10, JP4.10, R51.1
- net D2_B19: now also JP1.12, JP4.12, R52.1
- net D2_B2: now also JP1.9, JP4.9, R35.1
- net D2_B20: now also JP1.14, JP4.14, R53.1
- net D2_B21: now also JP1.16, JP4.16, R54.1
- net D2_B22: now also JP1.18, JP4.18, R55.1
- net D2_B23: now also JP1.20, JP4.20, R56.1, R58.1
- net D2_B24: now also JP1.22, JP4.22
- net D2_B25: now also JP1.24, JP4.24, R57.1
- net D2_B26: now also JP1.26, JP4.26, R59.1
- net D2_B27: now also JP1.28, JP4.28, R60.1
- net D2_B28: now also JP1.30, JP4.30, R61.1
- net D2_B29: now also JP1.32, JP1.34, JP4.32, JP4.34, R62.1
- net D2_B3: now also JP1.11, JP4.11, R36.1
- net D2_B30: now also R63.1
- net D2_B31: now also JP1.36, JP4.36, R64.1
- net D2_B4: now also JP1.13, JP4.13, R37.1
- net D2_B5: now also JP1.15, JP4.15, R38.1
- net D2_B6: now also JP1.17, JP4.17, R39.1
- net D2_B7: now also JP1.19, JP4.19, R40.1
- net D2_B8: now also JP1.21, JP4.21, R41.1
- net D2_B9: now also JP1.23, JP4.23, R42.1
- net GND: now also JP1.3, JP1.37, JP1.38, JP1.4, JP2.3, JP2.37, JP2.38, JP2.4, JP3.3, JP3.37, JP3.38, JP3.4, JP4.3, JP4.37, JP4.38, JP4.4, JP5.3, JP5.37, JP5.38, JP5.4, JP6.3, JP6.37, JP6.38, JP6.4, R1.2, R10.2, R11.2, R12.2, R13.2, R14.2, R15.2, R16.2, R17.2, R18.2, R19.2, R2.2, R20.2, R21.2, R22.2, R23.2, R24.2, R25.2, R26.2, R27.2, R28.2, R29.2, R3.2, R30.2, R31.2, R32.2, R33.2, R34.2, R35.2, R36.2, R37.2, R38.2, R39.2, R4.2, R40.2, R41.2, R42.2, R43.2, R44.2, R45.2, R46.2, R47.2, R48.2, R49.2, R5.2, R50.2, R51.2, R52.2, R53.2, R54.2, R55.2, R56.2, R57.2, R58.2, R59.2, R6.2, R60.2, R61.2, R62.2, R63.2, R64.2, R7.2, R8.2, R9.2; no longer R1.1, R10.1, R11.1, R12.1, R13.1, R14.1, R15.1, R16.1, R2.1, R3.1, R4.1, R5.1, R6.1, R7.1, R8.1, R9.1
- net SUM_B1: now also JP5.7, JP6.7
- net SUM_B10: now also JP5.25, JP6.25
- net SUM_B11: now also JP5.27, JP6.27
- net SUM_B12: now also JP5.29, JP6.29
- net SUM_B13: now also JP5.31, JP6.31
- net SUM_B14: now also JP5.33, JP6.33
- net SUM_B15: now also JP5.35, JP6.35
- net SUM_B16: now also JP5.6, JP6.6
- net SUM_B17: now also JP5.8, JP6.8
- net SUM_B18: now also JP5.10, JP6.10
- net SUM_B19: now also JP5.12, JP6.12
- net SUM_B2: now also JP5.9, JP6.9
- net SUM_B20: now also JP5.14, JP6.14
- net SUM_B21: now also JP5.16, JP6.16
- net SUM_B22: now also JP5.18, JP6.18
- net SUM_B23: now also JP5.20, JP6.20
- net SUM_B24: now also JP5.22, JP6.22
- net SUM_B25: now also JP5.24, JP6.24
- net SUM_B26: now also JP5.26, JP6.26
- net SUM_B27: now also JP5.28, JP6.28
- net SUM_B28: now also JP5.30, JP6.30
- net SUM_B29: now also JP5.32, JP5.34, JP6.32, JP6.34
- net SUM_B3: now also JP5.11, JP6.11
- net SUM_B31: now also JP5.36, JP6.36
- net SUM_B4: now also JP5.13, JP5.15, JP6.13, JP6.15
- net SUM_B6: now also JP5.17, JP6.17
- net SUM_B7: now also JP5.19, JP6.19
- net SUM_B8: now also JP5.21, JP6.21
- net SUM_B9: now also JP5.23, JP6.23

Commit message: Rename ALU Header Pins
Parts:
- moved IC47 531.8 mm to (-165.1, -416.6)
- moved IC45 525.7 mm to (-165.1, -406.4)
- moved IC43 521.3 mm to (-165.1, -396.2)
- moved IC41 518.5 mm to (-165.1, -386.1)
- moved IC48 514.7 mm to (-151.1, -375.9)
- moved IC46 481.4 mm to (-151.1, -365.8)
- moved IC44 475.7 mm to (-151.1, -355.6)
- moved IC42 471.9 mm to (-151.1, -345.4)
- moved JP3 165.1 mm to (-147.3, -281.9)
- moved JP4 157.5 mm to (-147.3, -289.6)
- moved JP6 149.9 mm to (-147.3, -297.2)
- moved R45 63.5 mm to (-163.8, -316.2)
- moved R46 63.5 mm to (-146.1, -316.2)
- moved R33 63.5 mm to (-163.8, -301.0)
- moved R34 63.5 mm to (-146.1, -301.0)
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Connections:
- removed net D1_B0: JP2.5, JP3.5, R1.1
- removed net D2_B0: JP1.5, JP4.5, R33.1
- removed net SUM_B0: JP5.5, JP6.5
- new net AND1_B33: IC47.9
- net AND1_B32: no longer IC47.9
- net D1_B1: now also JP2.5, JP3.5, R1.1; no longer JP2.7, JP3.7, R2.1
- net D1_B10: now also JP2.23, JP3.23, R10.1; no longer JP2.25, JP3.25, R11.1, R12.1
- net D1_B11: now also JP2.25, JP3.25, R11.1, R12.1; no longer JP2.27, JP3.27
- net D1_B12: now also JP2.27, JP3.27; no longer JP2.29, JP3.29, R13.1
- net D1_B13: now also JP2.29, JP3.29, R13.1; no longer JP2.31, JP3.31, R14.1
- net D1_B14: now also JP2.31, JP3.31, R14.1; no longer JP2.33, JP3.33, R15.1
- net D1_B15: now also JP2.33, JP3.33, R15.1; no longer JP2.35, JP3.35, R17.1
- net D1_B16: now also JP2.35, JP3.35, R17.1; no longer JP2.6, JP3.6, R16.1
- net D1_B17: now also JP2.6, JP3.6, R16.1; no longer JP2.8, JP3.8, R18.1
- net D1_B18: now also JP2.8, JP3.8, R18.1; no longer JP2.10, JP3.10, R19.1
- net D1_B19: now also JP2.10, JP3.10, R19.1; no longer JP2.12, JP3.12, R20.1
- net D1_B2: now also JP2.7, JP3.7, R2.1; no longer JP2.9, JP3.9, R3.1
- net D1_B20: now also JP2.12, JP3.12, R20.1; no longer JP2.14, JP3.14, R21.1
- net D1_B21: now also JP2.14, JP3.14, R21.1; no longer JP2.16, JP3.16, R22.1
- net D1_B22: now also JP2.16, JP3.16, R22.1; no longer JP2.18, JP3.18, R23.1
- net D1_B23: now also JP2.18, JP3.18, R23.1; no longer JP2.20, JP3.20, R24.1
- net D1_B24: now also JP2.20, JP3.20, R24.1; no longer JP2.22, JP3.22, R26.1
- net D1_B25: now also JP2.22, JP3.22, R26.1; no longer JP2.24, JP3.24, R25.1
- net D1_B26: now also JP2.24, JP3.24, R25.1; no longer JP2.26, JP3.26, R27.1
- net D1_B27: now also JP2.26, JP3.26, R27.1; no longer JP2.28, JP3.28, R28.1
- net D1_B28: now also JP2.28, JP3.28, R28.1; no longer JP2.30, JP3.30, R29.1
- net D1_B29: now also JP2.30, JP3.30, R29.1; no longer JP2.32, JP3.32, R30.1
- net D1_B3: now also JP2.9, JP3.9, R3.1; no longer JP2.11, JP3.11, R4.1
- net D1_B30: now also JP2.32, JP3.32, R30.1; no longer JP2.34, JP3.34, R31.1
- net D1_B31: now also JP2.34, JP3.34, R31.1; no longer JP2.36, JP3.36, R32.1
- net D1_B32: now also JP2.36, JP3.36, R32.1
- net D1_B4: now also JP2.11, JP3.11, R4.1; no longer JP2.13, JP3.13, R5.1
- net D1_B5: now also JP2.13, JP3.13, R5.1; no longer JP2.15, JP3.15, R6.1
- net D1_B6: now also JP2.15, JP3.15, R6.1; no longer JP2.17, JP3.17, R7.1
- net D1_B7: now also JP2.17, JP3.17, R7.1; no longer JP2.19, JP3.19, R8.1
- net D1_B8: now also JP2.19, JP3.19, R8.1; no longer JP2.21, JP3.21, R9.1
- net D1_B9: now also JP2.21, JP3.21, R9.1; no longer JP2.23, JP3.23, R10.1
- net D2_B1: now also JP1.5, JP4.5, R33.1; no longer JP1.7, JP4.7, R34.1
- net D2_B10: now also JP1.23, JP4.23, R42.1; no longer JP1.25, JP4.25, R43.1
- net D2_B11: now also JP1.25, JP4.25, R43.1; no longer JP1.27, JP4.27, R44.1
- net D2_B12: now also JP1.27, JP4.27, R44.1; no longer JP1.29, JP4.29, R45.1
- net D2_B13: now also JP1.29, JP4.29, R45.1; no longer JP1.31, JP4.31, R46.1
- net D2_B14: now also JP1.31, JP4.31, R46.1; no longer JP1.33, JP4.33, R47.1
- net D2_B15: now also JP1.33, JP4.33, R47.1; no longer JP1.35, JP4.35, R49.1
- net D2_B16: now also JP1.35, JP4.35, R49.1; no longer JP1.6, JP4.6, R48.1
- net D2_B17: now also JP1.6, JP4.6, R48.1; no longer JP1.8, JP4.8, R50.1
- net D2_B18: now also JP1.8, JP4.8, R50.1; no longer JP1.10, JP4.10, R51.1
- net D2_B19: now also JP1.10, JP4.10, R51.1; no longer JP1.12, JP4.12, R52.1
- net D2_B2: now also JP1.7, JP4.7, R34.1; no longer JP1.9, JP4.9, R35.1
- net D2_B20: now also JP1.12, JP4.12, R52.1; no longer JP1.14, JP4.14, R53.1
- net D2_B21: now also JP1.14, JP4.14, R53.1; no longer JP1.16, JP4.16, R54.1
- net D2_B22: now also JP1.16, JP4.16, R54.1; no longer JP1.18, JP4.18, R55.1
- net D2_B23: now also JP1.18, JP4.18, R55.1; no longer JP1.20, JP4.20, R56.1, R58.1
- net D2_B24: now also JP1.20, JP4.20, R56.1, R58.1; no longer JP1.22, JP4.22
- net D2_B25: now also JP1.22, JP4.22; no longer JP1.24, JP4.24, R57.1
- net D2_B26: now also JP1.24, JP4.24, R57.1; no longer JP1.26, JP4.26, R59.1
- net D2_B27: now also JP1.26, JP4.26, R59.1; no longer JP1.28, JP4.28, R60.1
- net D2_B28: now also JP1.28, JP4.28, R60.1; no longer JP1.30, JP4.30, R61.1
- net D2_B29: now also JP1.30, JP4.30, R61.1; no longer JP1.32, JP1.34, JP4.32, JP4.34, R62.1
- net D2_B3: now also JP1.9, JP4.9, R35.1; no longer JP1.11, JP4.11, R36.1
- net D2_B30: now also JP1.32, JP1.34, JP4.32, JP4.34, R62.1; no longer R63.1
- net D2_B31: now also R63.1; no longer JP1.36, JP4.36, R64.1
- net D2_B32: now also JP1.36, JP4.36, R64.1
- net D2_B4: now also JP1.11, JP4.11, R36.1; no longer JP1.13, JP4.13, R37.1
- net D2_B5: now also JP1.13, JP4.13, R37.1; no longer JP1.15, JP4.15, R38.1
- net D2_B6: now also JP1.15, JP4.15, R38.1; no longer JP1.17, JP4.17, R39.1
- net D2_B7: now also JP1.17, JP4.17, R39.1; no longer JP1.19, JP4.19, R40.1
- net D2_B8: now also JP1.19, JP4.19, R40.1; no longer JP1.21, JP4.21, R41.1
- net D2_B9: now also JP1.21, JP4.21, R41.1; no longer JP1.23, JP4.23, R42.1
- net SUM_B1: now also JP5.5, JP6.5; no longer JP5.7, JP6.7
- net SUM_B10: now also JP5.23, JP6.23; no longer JP5.25, JP6.25
- net SUM_B11: now also JP5.25, JP6.25; no longer JP5.27, JP6.27
- net SUM_B12: now also JP5.27, JP6.27; no longer JP5.29, JP6.29
- net SUM_B13: now also JP5.29, JP6.29; no longer JP5.31, JP6.31
- net SUM_B14: now also JP5.31, JP6.31; no longer JP5.33, JP6.33
- net SUM_B15: now also JP5.33, JP6.33; no longer JP5.35, JP6.35
- net SUM_B16: now also JP5.35, JP6.35; no longer JP5.6, JP6.6
- net SUM_B17: now also JP5.6, JP6.6; no longer JP5.8, JP6.8
- net SUM_B18: now also JP5.8, JP6.8; no longer JP5.10, JP6.10
- net SUM_B19: now also JP5.10, JP6.10; no longer JP5.12, JP6.12
- net SUM_B2: now also JP5.7, JP6.7; no longer JP5.9, JP6.9
- net SUM_B20: now also JP5.12, JP6.12; no longer JP5.14, JP6.14
- net SUM_B21: now also JP5.14, JP6.14; no longer JP5.16, JP6.16
- net SUM_B22: now also JP5.16, JP6.16; no longer JP5.18, JP6.18
- net SUM_B23: now also JP5.18, JP6.18; no longer JP5.20, JP6.20
- net SUM_B24: now also JP5.20, JP6.20; no longer JP5.22, JP6.22
- net SUM_B25: now also JP5.22, JP6.22; no longer JP5.24, JP6.24
- net SUM_B26: now also JP5.24, JP6.24; no longer JP5.26, JP6.26
- net SUM_B27: now also JP5.26, JP6.26; no longer JP5.28, JP6.28
- net SUM_B28: now also JP5.28, JP6.28; no longer JP5.30, JP6.30
- net SUM_B29: now also JP5.30, JP6.30; no longer JP5.32, JP5.34, JP6.32, JP6.34
- net SUM_B3: now also JP5.9, JP6.9; no longer JP5.11, JP6.11
- net SUM_B30: now also JP5.32, JP6.32
- net SUM_B31: now also JP5.34, JP6.34; no longer JP5.36, JP6.36
- net SUM_B32: now also JP5.36, JP6.36
- net SUM_B4: now also JP5.11, JP6.11; no longer JP5.13, JP5.15, JP6.13, JP6.15
- net SUM_B5: now also JP5.13, JP5.15, JP6.13, JP6.15
- net SUM_B6: no longer JP5.17, JP6.17
- net SUM_B7: now also JP5.17, JP6.17; no longer JP5.19, JP6.19
- net SUM_B8: now also JP5.19, JP6.19; no longer JP5.21, JP6.21
- net SUM_B9: now also JP5.21, JP6.21; no longer JP5.23, JP6.23

Commit message: Capacitors
Parts:
- added C1, C10, C11, C12, C13, C14, C15, C16, C17, C18, C19, C2, C20, C21, C22, C23, C24, C3, C4, C5, C6, C7, C8, C9: CC0603KRX7R9BB104, CC0603KRX7R9BB104:CAPC1608X90N
Connections:
- new net N$2: C1.2, C10.2, C11.2, C12.2, C13.2, C14.2, C15.2, C16.2, C17.2, C18.2, C19.2, C2.2, C20.2, C21.2, C22.2, C23.2, C24.2, C3.2, C4.2, C5.2, C6.2, C7.2, C8.2, C9.2
- net GND: now also C1.1, C10.1, C11.1, C12.1, C13.1, C14.1, C15.1, C16.1, C17.1, C18.1, C19.1, C2.1, C20.1, C21.1, C22.1, C23.1, C24.1, C3.1, C4.1, C5.1, C6.1, C7.1, C8.1, C9.1

Commit message: Resistors
Parts:
- moved C22 618.6 mm to (-22.9, 118.1)
- moved C23 615.7 mm to (-43.2, 118.1)
- moved C24 613.5 mm to (-63.5, 118.1)
- moved C16 601.5 mm to (-22.9, 115.6)
- moved C17 598.5 mm to (-43.2, 115.6)
- moved C18 596.2 mm to (-63.5, 115.6)
- moved C19 594.6 mm to (-83.8, 115.6)
- moved C20 593.6 mm to (-104.1, 115.6)
- moved C21 593.4 mm to (-124.5, 115.6)
- moved C10 584.5 mm to (-22.9, 113.0)
- moved C11 581.3 mm to (-43.2, 113.0)
- moved C12 578.9 mm to (-63.5, 113.0)
- moved C13 577.1 mm to (-83.8, 113.0)
- moved C14 576.1 mm to (-104.1, 113.0)
- moved C15 575.8 mm to (-124.5, 113.0)
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Connections:
- removed net N$1: IC1.7
- removed net N$106: IC8.14
- removed net N$113: IC9.7
- removed net N$120: IC9.14
- removed net N$127: IC10.7
- removed net N$134: IC10.14
- removed net N$141: IC11.7
- removed net N$148: IC11.14
- removed net N$15: IC2.7
- removed net N$155: IC12.7
- removed net N$162: IC12.14
- removed net N$169: IC13.7
- removed net N$176: IC13.14
- removed net N$183: IC14.7
- removed net N$190: IC14.14
- removed net N$197: IC15.7
- removed net N$204: IC15.14
- removed net N$211: IC16.7
- removed net N$218: IC16.14
- removed net N$22: IC2.14
- removed net N$231: IC33.7
- removed net N$238: IC33.14
- removed net N$245: IC34.7
- removed net N$252: IC34.14
- removed net N$259: IC35.7
- removed net N$266: IC35.14
- removed net N$273: IC36.7
- removed net N$280: IC36.14
- removed net N$287: IC37.7
- removed net N$294: IC37.14
- removed net N$3: IC3.14
- removed net N$301: IC38.7
- removed net N$308: IC38.14
- removed net N$315: IC39.7
- removed net N$329: IC40.7
- removed net N$336: IC40.14
- removed net N$343: IC41.7
- removed net N$344: IC41.14
- removed net N$345: IC17.7
- removed net N$352: IC17.14
- removed net N$359: IC18.7
- removed net N$366: IC18.14
- removed net N$373: IC19.7
- removed net N$380: IC19.14
- removed net N$387: IC20.7
- removed net N$394: IC20.14
- removed net N$401: IC21.7
- removed net N$408: IC21.14
- removed net N$415: IC22.7
- removed net N$422: IC22.14
- removed net N$429: IC23.7
- removed net N$43: IC4.7
- removed net N$436: IC23.14
- removed net N$443: IC24.7
- removed net N$450: IC24.14
- removed net N$463: IC25.7
- removed net N$470: IC25.14
- removed net N$477: IC26.7
- removed net N$484: IC26.14
- removed net N$491: IC27.7
- removed net N$498: IC27.14
- removed net N$50: IC4.14
- removed net N$505: IC28.7
- removed net N$512: IC28.14
- removed net N$519: IC29.7
- removed net N$526: IC29.14
- removed net N$533: IC30.7
- removed net N$540: IC30.14
- removed net N$547: IC31.7
- removed net N$554: IC31.14
- removed net N$561: IC32.7
- removed net N$568: IC32.14
- removed net N$57: IC5.7
- removed net N$64: IC5.14
- removed net N$701: IC42.7
- removed net N$702: IC42.14
- removed net N$71: IC6.7
- removed net N$715: IC43.7
- removed net N$716: IC43.14
- removed net N$729: IC44.7
- removed net N$730: IC44.14
- removed net N$743: IC45.7
- removed net N$744: IC45.14
- removed net N$757: IC46.7
- removed net N$758: IC46.14
- removed net N$771: IC47.7
- removed net N$772: IC47.14
- removed net N$78: IC6.14
- removed net N$785: IC48.7
- removed net N$786: IC48.14
- removed net N$8: IC1.14
- removed net N$85: IC7.7
- removed net N$92: IC7.14
- removed net N$99: IC8.7
- net D1_B11: no longer R12.1
- net D1_B12: now also R12.1
- net D1_B15: no longer IC39.14
- net D2_B24: no longer R58.1
- net D2_B25: now also R58.1
- net D2_B30: no longer JP1.34, JP4.34
- net D2_B31: now also JP1.34, JP4.34
- net GND: now also IC1.7, IC10.7, IC11.7, IC12.7, IC13.7, IC14.7, IC15.7, IC16.7, IC17.7, IC18.7, IC19.7, IC2.7, IC20.7, IC21.7, IC22.7, IC23.7, IC24.7, IC25.7, IC26.7, IC27.7, IC28.7, IC29.7, IC3.7, IC30.7, IC31.7, IC32.7, IC33.7, IC34.7, IC35.7, IC36.7, IC37.7, IC38.7, IC39.7, IC4.7, IC40.7, IC41.7, IC42.7, IC43.7, IC44.7, IC45.7, IC46.7, IC47.7, IC48.7, IC5.7, IC6.7, IC7.7, IC8.7, IC9.7
- net SUM_B5: no longer JP5.15, JP6.15
- net SUM_B6: now also JP5.15, JP6.15
- net VCC: now also IC1.14, IC10.14, IC11.14, IC12.14, IC13.14, IC14.14, IC15.14, IC16.14, IC17.14, IC18.14, IC19.14, IC2.14, IC20.14, IC21.14, IC22.14, IC23.14, IC24.14, IC25.14, IC26.14, IC27.14, IC28.14, IC29.14, IC3.14, IC30.14, IC31.14, IC32.14, IC33.14, IC34.14, IC35.14, IC36.14, IC37.14, IC38.14, IC39.14, IC4.14, IC40.14, IC41.14, IC42.14, IC43.14, IC44.14, IC45.14, IC46.14, IC47.14, IC48.14, IC5.14, IC6.14, IC7.14, IC8.14, IC9.14
- net XOR_B6: no longer IC3.7
Routing:
- net VCC: track 0.00 -> 1.75 mm
Other:
- board size 98.7 x 99 mm -> 97.8 x 98.7 mm

Commit message: Alu design
Parts:
- moved R63 206.5 mm to (81.3, 14.0), turned to 90 degrees
- moved C3 198.9 mm to (73.7, 45.7)
- moved R56 189.8 mm to (63.5, 14.0), turned to 90 degrees
- moved IC22 187.8 mm to (68.6, 40.6)
- moved IC14 176.5 mm to (58.4, 52.1)
- moved IC21 175.6 mm to (68.6, 29.2)
- moved C8 174.9 mm to (53.3, 34.3)
- moved C7 174.9 mm to (73.7, 34.3)
- moved R3 172.1 mm to (50.8, 85.1), turned to 270 degrees
- moved IC13 163.1 mm to (58.4, 63.5)
- moved IC12 158.8 mm to (68.6, 52.1)
- moved C15 157.2 mm to (29.2, 80.0)
- moved IC6 155.8 mm to (24.1, 86.4)
- moved C21 155.6 mm to (29.2, 91.4)
- moved C1 153.7 mm to (73.7, 68.6)
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Connections:
- removed net N$2: C1.2, C10.2, C11.2, C12.2, C13.2, C14.2, C15.2, C16.2, C17.2, C18.2, C19.2, C2.2, C20.2, C21.2, C22.2, C23.2, C24.2, C3.2, C4.2, C5.2, C6.2, C7.2, C8.2, C9.2
- removed net N$30: IC3.6
- net VCC: now also C1.2, C10.2, C11.2, C12.2, C13.2, C14.2, C15.2, C16.2, C17.2, C18.2, C19.2, C2.2, C20.2, C21.2, C22.2, C23.2, C24.2, C3.2, C4.2, C5.2, C6.2, C7.2, C8.2, C9.2
- net XOR_B6: now also IC3.6

Commit message: Modify ALU & Libraries
Parts:
- moved R64 249.9 mm to (-128.3, 146.1), turned to 0 degrees
- moved R57 234.3 mm to (-128.3, 141.0), turned to 0 degrees
- moved R63 232.9 mm to (-110.5, 146.1), turned to 0 degrees
- moved R43 228.1 mm to (-128.3, 130.8), turned to 0 degrees
- moved R49 226.3 mm to (-110.5, 135.9), turned to 0 degrees
- moved IC33 219.1 mm to (223.5, 35.6)
- moved IC25 218.8 mm to (223.5, 55.9)
- moved IC42 217.3 mm to (223.5, 45.7)
- moved R62 216.4 mm to (-92.7, 146.1), turned to 0 degrees
- moved R56 215.4 mm to (-110.5, 141.0), turned to 0 degrees
- moved R50 214.5 mm to (-128.3, 135.9), turned to 0 degrees
- moved R15 211.1 mm to (-128.3, 110.5), turned to 0 degrees
- moved R42 210.7 mm to (-110.5, 130.8), turned to 0 degrees
- moved R36 210.2 mm to (-128.3, 125.7), turned to 0 degrees
- moved IC1 207.2 mm to (213.4, 66.0)
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Connections:
- removed net AND1_B33: IC47.9
- net AND1_B32: now also IC47.9
Routing:
- net AND1_B2: track 0.00 -> 18.6 mm
- net AND1_B1: track 0.00 -> 15.6 mm
- net AND1_B3: track 0.00 -> 14.2 mm
- net AND1_B4: track 0.00 -> 14.0 mm
- net AND2_B1: track 0.00 -> 13.4 mm
- net AND2_B2: track 0.00 -> 12.6 mm
- net INV_B1: track 0.00 -> 10.5 mm
- net INV_B2: track 0.00 -> 9.88 mm
- net XOR_B4: track 0.00 -> 9.79 mm
- net XOR_B3: track 0.00 -> 9.72 mm
- net SUM_B1: track 0.00 -> 9.43 mm
- net AND2_B3: track 0.00 -> 9.41 mm
- net AND2_B4: track 0.00 -> 9.28 mm
- net XOR_B1: track 0.00 -> 9.26 mm
- net XOR_B2: track 0.00 -> 8.61 mm
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Other:
- board size 97.8 x 98.7 mm -> 160 x 100 mm
